Commit message: edit mybot into agv_lidar

File: description/robot_core.xacro (robot description, xacro)
@@ -5,6 +5,6 @@
         <color rgba="1 1 1 1" />
     </material>
-    <material name="orange">
-        <color rgba="1 0.3 0.1 1"/>
+    <material name="red">
+        <color rgba="1 0.2 0.2 1"/>
     </material>
     <material name="blue">
@@ -15,35 +15,35 @@
     </material>
     <!-- BASE LINK -->
-    <link name="base_link">
+    <link name="robot_base">
     </link>
     <!-- CHASSIS LINK -->
     <joint name="chassis_joint" type="fixed">
-        <parent link="base_link"/>
+        <parent link="robot_base"/>
         <child link="chassis"/>
-        <origin xyz="-0.1 0 0"/>
+        <origin xyz="-0.25 0 0"/>
     </joint>
     <link name="chassis">
         <visual>
-            <origin xyz="0.15 0 0.075"/>
+            <origin xyz="0.25 0 0.1"/>
             <geometry>
-                <box size="0.3 0.3 0.15"/>
+                <box size="0.5 0.5 0.2"/>
             </geometry>
             <material name="white"/>
         </visual>
         <collision>
-            <origin xyz="0.15 0 0.075"/>
+            <origin xyz="0.25 0 0.1"/>
             <geometry>
-                <box size="0.3 0.3 0.15"/>
+                <box size="0.5 0.5 0.2"/>
             </geometry>
         </collision>
-        <xacro:inertial_box mass="0.5" x="0.3" y="0.3" z="0.15">
-            <origin xyz="0.15 0 0.075" rpy="0 0 0"/>
+        <xacro:inertial_box mass="0.5" x="0.5" y="0.5" z="0.2">
+            <origin xyz="0.25 0 0.1" rpy="0 0 0"/>
         </xacro:inertial_box>
     </link>
     <!-- LEFT WHEEL LINK -->
     <joint name="left_wheel_joint" type="continuous">
-        <parent link="base_link"/>
+        <parent link="robot_base"/>
         <child link="left_wheel"/>
-        <origin xyz="0 0.175 0" rpy="-${pi/2} 0 0" />
+        <origin xyz="0 0.25 0" rpy="-${pi/2} 0 0" />
         <axis xyz="0 0 1"/>
     </joint>
@@ -51,14 +51,14 @@
         <visual>
             <geometry>
-                <cylinder radius="0.05" length="0.04"/>
+                <cylinder radius="0.1" length="0.03"/>
             </geometry>
-            <material name="blue"/>
+            <material name="red"/>
         </visual>
         <collision>
             <geometry>
-                <cylinder radius="0.05" length="0.04"/>
+                <cylinder radius="0.1" length="0.03"/>
             </geometry>
         </collision>
-        <xacro:inertial_cylinder mass="0.1" length="0.04" radius="0.05">
+        <xacro:inertial_cylinder mass="0.1" radius="0.1" length="0.03">
             <origin xyz="0 0 0" rpy="0 0 0"/>
         </xacro:inertial_cylinder>
@@ -66,5 +66,5 @@
     <!-- RIGHT WHEEL LINK -->
     <joint name="right_wheel_joint" type="continuous">
-        <parent link="base_link"/>
+        <parent link="robot_base"/>
         <child link="right_wheel"/>
         <origin xyz="0 -0.175 0" rpy="${pi/2} 0 0" />
@@ -74,24 +74,45 @@
         <visual>
             <geometry>
-                <cylinder radius="0.05" length="0.04"/>
+                <cylinder radius="0.1" length="0.03"/>
             </geometry>
-            <material name="blue"/>
+            <material name="red"/>
         </visual>
         <collision>
             <geometry>
-                <cylinder radius="0.05" length="0.04"/>
+                <cylinder radius="0.1" length="0.03"/>
             </geometry>
         </collision>
-        <xacro:inertial_cylinder mass="0.1" length="0.04" radius="0.05">
+        <xacro:inertial_cylinder mass="0.1" radius="0.1" length="0.03">
             <origin xyz="0 0 0" rpy="0 0 0"/>
         </xacro:inertial_cylinder>
     </link>
     <!-- CASTER WHEEL LINK -->
-    <joint name="caster_wheel_joint" type="fixed">
+    <joint name="caster_wheel_f_joint" type="fixed">
         <parent link="chassis"/>
-        <child link="caster_wheel"/>
-        <origin xyz="0.24 0 0"/>
+        <child link="caster_wheel_f"/>
+        <origin xyz="0.4 0 0"/>
     </joint>
-    <link name="caster_wheel">
+    <link name="caster_wheel_f">
+        <visual>
+            <geometry>
+                <sphere radius="0.05"/>
+            </geometry>
+            <material name="black"/>
+        </visual>
+        <collision>
+            <geometry>
+                <sphere radius="0.05"/>
+            </geometry>
+        </collision>
+        <xacro:inertial_sphere mass="0.1" radius="0.05">
+            <origin xyz="0 0 0" rpy="0 0 0"/>
+        </xacro:inertial_sphere>
+    </link>
+    <joint name="caster_wheel_b_joint" type="fixed">
+        <parent link="chassis"/>
+        <child link="caster_wheel_b"/>
+        <origin xyz="0.1 0 0"/>
+    </joint>
+    <link name="caster_wheel_b">
         <visual>
             <geometry>

Commit message: kendali robot in gazebo with keyboard(blm berhasil)

File: description/robot_core.xacro (robot description, xacro)
@@ -41,9 +41,12 @@
         </xacro:inertial_box>
     </link>
+    <gazebo reference="chassis">
+        <material>Gazebo/White</material>
+    </gazebo>
     <!-- LEFT WHEEL LINK -->
     <joint name="left_wheel_joint" type="continuous">
         <parent link="robot_base"/>
         <child link="left_wheel"/>
-        <origin xyz="0 0.25 0" rpy="-${pi/2} 0 0" />
+        <origin xyz="0 0.175 -0.03" rpy="-${pi/2} 0 0" />
         <axis xyz="0 0 1"/>
     </joint>
@@ -51,5 +54,5 @@
         <visual>
             <geometry>
-                <cylinder radius="0.1" length="0.03"/>
+                <cylinder radius="0.05" length="0.03"/>
             </geometry>
             <material name="red"/>
@@ -57,16 +60,19 @@
         <collision>
             <geometry>
-                <cylinder radius="0.1" length="0.03"/>
+                <cylinder radius="0.05" length="0.03"/>
             </geometry>
         </collision>
-        <xacro:inertial_cylinder mass="0.1" radius="0.1" length="0.03">
+        <xacro:inertial_cylinder mass="0.1" radius="0.05" length="0.03">
             <origin xyz="0 0 0" rpy="0 0 0"/>
         </xacro:inertial_cylinder>
     </link>
+    <gazebo reference="left_wheel">
+        <material>Gazebo/Red</material>
+    </gazebo>
     <!-- RIGHT WHEEL LINK -->
     <joint name="right_wheel_joint" type="continuous">
         <parent link="robot_base"/>
         <child link="right_wheel"/>
-        <origin xyz="0 -0.175 0" rpy="${pi/2} 0 0" />
+        <origin xyz="0 -0.175 -0.03" rpy="${pi/2} 0 0" />
         <axis xyz="0 0 -1"/>
     </joint>
@@ -74,5 +80,5 @@
         <visual>
             <geometry>
-                <cylinder radius="0.1" length="0.03"/>
+                <cylinder radius="0.05" length="0.03"/>
             </geometry>
             <material name="red"/>
@@ -80,21 +86,24 @@
         <collision>
             <geometry>
-                <cylinder radius="0.1" length="0.03"/>
+                <cylinder radius="0.05" length="0.03"/>
             </geometry>
         </collision>
-        <xacro:inertial_cylinder mass="0.1" radius="0.1" length="0.03">
+        <xacro:inertial_cylinder mass="0.1" radius="0.05" length="0.03">
             <origin xyz="0 0 0" rpy="0 0 0"/>
         </xacro:inertial_cylinder>
     </link>
+    <gazebo reference="right_wheel">
+        <material>Gazebo/Red</material>
+    </gazebo>
     <!-- CASTER WHEEL LINK -->
     <joint name="caster_wheel_f_joint" type="fixed">
         <parent link="chassis"/>
         <child link="caster_wheel_f"/>
-        <origin xyz="0.4 0 0"/>
+        <origin xyz="0.4 0 -0.04"/>
     </joint>
     <link name="caster_wheel_f">
         <visual>
             <geometry>
-                <sphere radius="0.05"/>
+                <sphere radius="0.04"/>
             </geometry>
             <material name="black"/>
@@ -102,20 +111,26 @@
         <collision>
             <geometry>
-                <sphere radius="0.05"/>
+                <sphere radius="0.04"/>
             </geometry>
         </collision>
-        <xacro:inertial_sphere mass="0.1" radius="0.05">
+        <xacro:inertial_sphere mass="0.1" radius="0.04">
             <origin xyz="0 0 0" rpy="0 0 0"/>
         </xacro:inertial_sphere>
     </link>
+    <gazebo reference="caster_wheel_f">
+        <material>Gazebo/Black</material>
+        <mu1 value="0.001"/>
+        <mu2 value="0.001"/>
+    </gazebo>
+    <!-- CASTER WHEEL LINK -->
     <joint name="caster_wheel_b_joint" type="fixed">
         <parent link="chassis"/>
         <child link="caster_wheel_b"/>
-        <origin xyz="0.1 0 0"/>
+        <origin xyz="0.1 0 -0.04"/>
     </joint>
     <link name="caster_wheel_b">
         <visual>
             <geometry>
-                <sphere radius="0.05"/>
+                <sphere radius="0.04"/>
             </geometry>
             <material name="black"/>
@@ -123,10 +138,15 @@
         <collision>
             <geometry>
-                <sphere radius="0.05"/>
+                <sphere radius="0.04"/>
             </geometry>
         </collision>
-        <xacro:inertial_sphere mass="0.1" radius="0.05">
+        <xacro:inertial_sphere mass="0.1" radius="0.04">
             <origin xyz="0 0 0" rpy="0 0 0"/>
         </xacro:inertial_sphere>
     </link>
+    <gazebo reference="caster_wheel_b">
+        <material>Gazebo/Black</material>
+        <mu1 value="0.001"/>
+        <mu2 value="0.001"/>
+    </gazebo>
 </robot>
