Commit message: kendali robot in gazebo with keyboard(berhasil)

File: description/kendali_gazebo.xacro (robot description, xacro)
@@ -9,6 +9,6 @@
             <wheel_diameter>0.1</wheel_diameter>
             <!-- limit -->
-            <max_wheel_torque>500</max_wheel_torque>
-            <max_wheel_acceleration>50.0</max_wheel_acceleration>
+            <max_wheel_torque>200</max_wheel_torque>
+            <max_wheel_acceleration>10.0</max_wheel_acceleration>
             <!-- output -->
             <odometry_frame>odom</odometry_frame>

File: description/robot.urdf.xacro (robot description, xacro)
@@ -2,3 +2,4 @@
 <robot xmlns:xacro="http://www.ros.org/wiki/xacro"  name="robot">
     <xacro:include filename="robot_core.xacro" />
+    <xacro:include filename="kendali_gazebo.xacro"/>
 </robot>

File: description/robot_core.xacro (robot description, xacro)
@@ -48,5 +48,5 @@
         <parent link="robot_base"/>
         <child link="left_wheel"/>
-        <origin xyz="0 0.175 -0.03" rpy="-${pi/2} 0 0" />
+        <origin xyz="0 0.2 0" rpy="-${pi/2} 0 0" />
         <axis xyz="0 0 1"/>
     </joint>
@@ -74,5 +74,5 @@
         <parent link="robot_base"/>
         <child link="right_wheel"/>
-        <origin xyz="0 -0.175 -0.03" rpy="${pi/2} 0 0" />
+        <origin xyz="0 -0.2 0" rpy="${pi/2} 0 0" />
         <axis xyz="0 0 -1"/>
     </joint>
@@ -100,10 +100,10 @@
         <parent link="chassis"/>
         <child link="caster_wheel_f"/>
-        <origin xyz="0.4 0 -0.04"/>
+        <origin xyz="0.4 0 0"/>
     </joint>
     <link name="caster_wheel_f">
         <visual>
             <geometry>
-                <sphere radius="0.04"/>
+                <sphere radius="0.05"/>
             </geometry>
             <material name="black"/>
@@ -111,8 +111,8 @@
         <collision>
             <geometry>
-                <sphere radius="0.04"/>
+                <sphere radius="0.05"/>
             </geometry>
         </collision>
-        <xacro:inertial_sphere mass="0.1" radius="0.04">
+        <xacro:inertial_sphere mass="0.1" radius="0.05">
             <origin xyz="0 0 0" rpy="0 0 0"/>
         </xacro:inertial_sphere>
@@ -127,10 +127,10 @@
         <parent link="chassis"/>
         <child link="caster_wheel_b"/>
-        <origin xyz="0.1 0 -0.04"/>
+        <origin xyz="0.1 0 0"/>
     </joint>
     <link name="caster_wheel_b">
         <visual>
             <geometry>
-                <sphere radius="0.04"/>
+                <sphere radius="0.05"/>
             </geometry>
             <material name="black"/>
@@ -138,8 +138,8 @@
         <collision>
             <geometry>
-                <sphere radius="0.04"/>
+                <sphere radius="0.05"/>
             </geometry>
         </collision>
-        <xacro:inertial_sphere mass="0.1" radius="0.04">
+        <xacro:inertial_sphere mass="0.1" radius="0.05">
             <origin xyz="0 0 0" rpy="0 0 0"/>
         </xacro:inertial_sphere>
